File: BOARD/TempControl/TempControl .brd (EAGLE design)
At the start: 100 x 80 mm, 21 parts, among them Q1 BD139, Q2 BD139, Q3 BD139, U1 ARDUINOR3-BPLACE

Commit message: miniors changes
Routing:
- added copper zone on layer 16, net GND
Other:
- board size 100 x 80 mm -> 73.7 x 55.9 mm
Changed lines of the file:
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@@
 <setting verticaltext="up"/>
 </settings>
-<grid distance="25" unitdist="mil" unit="mil" style="lines" multiple="2" display="yes" altdistance="25" altunitdist="mil" altunit="mil"/>
+<grid distance="50" unitdist="mil" unit="mil" style="lines" multiple="1" display="yes" altdistance="5" altunitdist="mil" altunit="mil"/>
 <layers>
 <layer number="1" name="Top" color="4" fill="1" visible="yes" active="yes"/>
@@
 <layer number="17" name="Pads" color="2" fill="1" visible="yes" active="yes"/>
 <layer number="18" name="Vias" color="2" fill="1" visible="yes" active="yes"/>
-<layer number="19" name="Unrouted" color="6" fill="1" visible="yes" active="yes"/>
+<layer number="19" name="Unrouted" color="6" fill="1" visible="no" active="yes"/>
 <layer number="20" name="Dimension" color="15" fill="1" visible="yes" active="yes"/>
 <layer number="21" name="tPlace" color="7" fill="1" visible="yes" active="yes"/>
 <layer number="22" name="bPlace" color="7" fill="1" visible="yes" active="yes"/>
-<layer number="23" name="tOrigins" color="15" fill="1" visible="yes" active="yes"/>
+<layer number="23" name="tOrigins" color="15" fill="1" visible="no" active="yes"/>
 <layer number="24" name="bOrigins" color="15" fill="1" visible="yes" active="yes"/>
 <layer number="25" name="tNames" color="7" fill="1" visible="yes" active="yes"/>
-<layer number="26" name="bNames" color="7" fill="1" visible="yes" active="yes"/>
-<layer number="27" name="tValues" color="7" fill="1" visible="yes" active="yes"/>
+<layer number="26" name="bNames" color="7" fill="1" visible="no" active="yes"/>
+<layer number="27" name="tValues" color="7" fill="1" visible="no" active="yes"/>
 <layer number="28" name="bValues" color="7" fill="1" visible="yes" active="yes"/>
 <layer number="29" name="tStop" color="7" fill="3" visible="no" active="yes"/>
@@
 <board>
 <plain>
-<wire x1="0" y1="0" x2="100" y2="0" width="0" layer="20"/>
-<wire x1="100" y1="0" x2="100" y2="80" width="0" layer="20"/>
-<wire x1="100" y1="80" x2="0" y2="80" width="0" layer="20"/>
-<wire x1="0" y1="80" x2="0" y2="0" width="0" layer="20"/>
+<wire x1="0" y1="0" x2="73.66" y2="0" width="0" layer="20"/>
+<wire x1="73.66" y1="0" x2="73.66" y2="55.88" width="0" layer="20"/>
+<wire x1="73.66" y1="55.88" x2="0" y2="55.88" width="0" layer="20"/>
+<wire x1="0" y1="55.88" x2="0" y2="0" width="0" layer="20"/>
 </plain>
 <attributes>
@@
 <wire x1="17.0434" y1="15.1892" x2="6.985" y2="17.6276" width="0" layer="19" extent="16-16"/>
 <wire x1="41.91" y1="31.75" x2="33.655" y2="38.1" width="0" layer="19" extent="16-16"/>
+<polygon width="0.8128" layer="16" isolate="0.8128">
+<vertex x="1.905" y="54.61"/>
+<vertex x="66.04" y="54.61"/>
+<vertex x="67.945" y="52.705"/>
+<vertex x="67.945" y="41.91"/>
+<vertex x="71.12" y="38.735"/>
+<vertex x="71.12" y="6.985"/>
+<vertex x="67.945" y="3.81"/>
+<vertex x="67.945" y="1.27"/>
+<vertex x="1.905" y="1.27"/>
+</polygon>
 </signal>
 <signal name="3V">
